File: PCB_Preamp_Power/untitled.kicad_sch (KiCad schematic)
At the start: 59 parts, among them SW1 SW_Push_DPDT

Commit message: PCBV3_Preamp_Power
Parts:
- added J2: Jack-DC, Preamp:CONN_NRJ4HF-1_NTK, symbol Connector:Jack-DC
- 12ax1, 12ax2, 12ax3, 12ax4: footprint (none) -> Preamp:NOVAL_BOTTOM_PCB
- C1, C10, C8, C9: footprint (none) -> Capacitor_SMD:C_0201_0603Metric
- C2, C20, C5: footprint (none) -> Library_f:Capa_L11mm_a2.5
- C21, C22, C24, C25, C26, C3, C4, C6, C7: footprint (none) -> Capacitor_SMD:C_0603_1608Metric
- C23: renamed from C13; footprint (none) -> Capacitor_SMD:C_0603_1608Metric
- Gain1_Post1: renamed from RV2; footprint (none) -> Connector_JST:JST_EH_B3B-EH-A_1x03_P2.50mm_Vertical
- Gain1_before1: renamed from RV1; footprint (none) -> Connector_JST:JST_EH_B3B-EH-A_1x03_P2.50mm_Vertical
- Gain2_Post1: renamed from RV7; footprint (none) -> Connector_JST:JST_EH_B3B-EH-A_1x03_P2.50mm_Vertical
- R1, R11, R2, R21, R22, R23, R25, R4, R5, R9: footprint (none) -> Resistor_SMD:R_0402_1005Metric
- R10, R12, R13, R24, R26, R27: footprint (none) -> Resistor_SMD:R_1206_3216Metric
- R14, R28: value 1.5k -> 2.2k; footprint (none) -> Resistor_SMD:R_1206_3216Metric
- R15, R16, R20, R29, R3, R30, R7, R8: footprint (none) -> Resistor_SMD:R_2010_5025Metric
- R6: footprint (none) -> Resistor_SMD:R_0805_2012Metric
- RV6: footprint (none) -> Connector_JST:JST_EH_B3B-EH-A_1x03_P2.50mm_Vertical
- SW1: footprint (none) -> Library_f:Holes_Switch_DPDT
- Vol1_high1: renamed from RV4; footprint (none) -> Connector_JST:JST_EH_B3B-EH-A_1x03_P2.50mm_Vertical
- Vol1_low2: renamed from RV5; footprint (none) -> Connector_JST:JST_EH_B3B-EH-A_1x03_P2.50mm_Vertical
- Vol2_high1: renamed from RV9; footprint (none) -> Connector_JST:JST_EH_B3B-EH-A_1x03_P2.50mm_Vertical
- Vol2_low1: renamed from RV10; footprint (none) -> Connector_JST:JST_EH_B3B-EH-A_1x03_P2.50mm_Vertical
- tone1: renamed from RV3; footprint (none) -> Connector_JST:JST_EH_B3B-EH-A_1x03_P2.50mm_Vertical
- tone2: renamed from RV8; footprint (none) -> Connector_JST:JST_EH_B3B-EH-A_1x03_P2.50mm_Vertical
Connections:
- net 6: no longer Vol2_low1.2
- net at R1.1, R2.2: now also J2.1
- net at R11.2, R12.2, R14.1: now also R13.1
- net at R25.2, R26.2, R28.1: now also R27.1
- net neutre: now reaches SW1.5 (B)
- net neutre: now also J2.2
- new net 10: Vol2_low1.2
Other:
- moved on the sheet: C25, C9, R1, R2
